File: esp32/esp32.kicad_sch (KiCad schematic)
At the start: 2 parts, among them U1 ESP32-S3

Commit message: done with full project
Parts:
- removed U1: ESP32-S3, Package_DFN_QFN:QFN-56-1EP_7x7mm_P0.4mm_EP4x4mm, symbol MCU_Espressif:ESP32-S3
- added C1, C2: 10uF, Capacitor_SMD:C_0805_2012Metric_Pad1.18x1.45mm_HandSolder, symbol Device:C
- added C3, C4: 0.1uF, Capacitor_SMD:C_0603_1608Metric_Pad1.08x0.95mm_HandSolder, symbol Device:C
- added C5: 10uF, Capacitor_SMD:C_0603_1608Metric_Pad1.08x0.95mm_HandSolder, symbol Device:C
- added C6: 1u, Capacitor_SMD:C_0603_1608Metric_Pad1.08x0.95mm_HandSolder, symbol Device:C
- added C7, C8: .1u, Capacitor_SMD:C_0603_1608Metric_Pad1.08x0.95mm_HandSolder, symbol Device:C
- added D2, D4: SC4340L-01ETG, Diode_SMD:D_0603_1608Metric_Pad1.05x0.95mm_HandSolder, symbol Device:D_TVS
- added D3: SS14, Diode_SMD:D_SMA, symbol Diode:SS14
- added J1: USB_C_Receptacle_USB2.0_16P, Connector_USB:USB_C_Receptacle_G-Switch_GT-USB-7010ASV, symbol Connector:USB_C_Receptacle_USB2.0_16P
- added J2: Conn_01x04_Pin, Connector_PinSocket_2.54mm:PinSocket_1x04_P2.54mm_Vertical, symbol Connector:Conn_01x04_Pin
- added R1, R2: 5.1k, Resistor_SMD:R_0603_1608Metric_Pad0.98x0.95mm_HandSolder, symbol Device:R
- added R3: 1k, Resistor_SMD:R_0603_1608Metric_Pad0.98x0.95mm_HandSolder, symbol Device:R
- added R4: 10k, Resistor_SMD:R_0603_1608Metric_Pad0.98x0.95mm_HandSolder, symbol Device:R
- added R5, R6: 4.7k, Resistor_SMD:R_0603_1608Metric_Pad0.98x0.95mm_HandSolder, symbol Device:R
- added SW1: SW_Push_Open, Button_Switch_SMD:SW_Push_1P1T_NO_CK_KMR2, symbol Switch:SW_Push_Open
- added TP1: TestPoint, TestPoint:TestPoint_Keystone_5010-5014_Multipurpose, symbol Connector:TestPoint
- added U1: ESP32-S3-WROOM-1, RF_Module:ESP32-S3-WROOM-1, symbol RF_Module:ESP32-S3-WROOM-1
- added U2: AP2112K-3.3, Package_TO_SOT_SMD:SOT-23-5, symbol Regulator_Linear:AP2112K-3.3
- added U3: BME280, Package_LGA:Bosch_LGA-8_2.5x2.5mm_P0.65mm_ClockwisePinNumbering, symbol Sensor:BME280
- D1: footprint (none) -> LED_SMD:LED_0603_1608Metric_Pad1.05x0.95mm_HandSolder
Connections:
- net GND: now also D1.1 (K), C1.2, C2.2, C3.2, C4.2, C5.2, C6.2, C7.2, C8.2, D2.1 (A1), D4.1 (A1), J1.A1 (GND), J1.A12 (GND), J1.B1 (GND), J1.B12 (GND), J1.S1 (SHIELD), J2.4 (Pin_4), R1.2, R2.2, SW1.2 (B), U1.1 (GND), U1.40 (GND), U1.41 (GND), U2.2 (GND), U3.1 (GND), U3.5 (SDO), U3.7 (GND)
- net at D1.2 (A): now also R3.1
- new net: R3.2, U1.4 (IO4)
- new net: J1.A5 (CC1), R1.1
- new net: J1.B5 (CC2), R2.1
- new net: C1.1, C3.1, D3.1 (K), U2.1 (VIN), U2.3 (EN)
- new net: TP1.1, U1.27 (IO0)
- new net +3.3V: C2.1, C4.1, C5.1, C7.1, C8.1, J2.1 (Pin_1), R4.1, R5.1, R6.1, U1.2 (3V3), U2.5 (VOUT), U3.2 (CSB), U3.6 (VDDIO), U3.8 (VDD)
- new net EN: C6.1, R4.2, SW1.1 (A), U1.3 (EN)
- new net RXD0: J2.3 (Pin_3), U1.36 (RXD0)
- new net SCK: R5.2, U1.17 (IO9), U3.4 (SCK)
- new net SDI: R6.2, U1.12 (IO8), U3.3 (SDI)
- new net TXD0: J2.2 (Pin_2), U1.37 (TXD0)
- new net VBUS: D3.2 (A), J1.A4 (VBUS), J1.A9 (VBUS), J1.B4 (VBUS), J1.B9 (VBUS)
- new net d+: D4.2 (A2), J1.A6 (D+), J1.B6 (D+), U1.14 (USB_D+)
- new net d-: D2.2 (A2), J1.A7 (D-), J1.B7 (D-), U1.13 (USB_D-)
- no-connect marks 0 -> 30
Other:
- note added: "A direct connection between SCB and VDDIO is Required"
- note added: "Connection Header"
- note added: "ESD protection diodes"
- note added: "Power Supply"
- note added: "Required Sensor - Pressure/Humidity"
- note added: "SDO tied to GND to select I2C address"
- moved on the sheet: D1
